Commit message: improved

File: Dexter/install/dexter_description/share/dexter_description/urdf/dexter.urdf.xacro (robot description, xacro)
@@ -1 +1,238 @@
-/home/aditya/Cpps/Dexter/dexter_description/urdf/dexter.urdf.xacro
+<?xml version="1.0"?>
+<robot xmlns:xacro="http://www.ros.org/wiki/xacro" name="dexter">
+    <xacro:arg name="is_ignition" default="true"/>
+    <xacro:arg name="is_sim"      default="true"/>
+    <xacro:include filename="$(find dexter_description)/urdf/dexter_gazebo.xacro" />
+    <xacro:include filename="$(find dexter_description)/urdf/dexter_ros2_control.xacro" />
+    <xacro:property name="PI"       value="3.14159265359" />
+    <xacro:property name="effort"   value="30.0" />
+    <xacro:property name="velocity" value="10.0" />
+    <xacro:macro name="default_inertial" params="mass">
+        <inertial>
+            <origin xyz="0 0 0" rpy="0 0 0"/>
+            <mass value="${mass}" />
+            <inertia ixx="1.0" ixy="0.0" ixz="0.0"
+                     iyy="1.0" iyz="0.0"
+                     izz="1.0" />
+        </inertial>
+    </xacro:macro>
+    <!-- ── Links ──────────────────────────────────────────────────────────── -->
+    <link name="world"/>
+    <link name="base_link">
+        <xacro:default_inertial mass="1.0"/>
+        <visual>
+            <origin rpy="0 0 0" xyz="-0.5 -0.5 0"/>
+            <geometry>
+                <mesh filename="package://dexter_description/meshes/basement.STL"
+                      scale="0.01 0.01 0.01"/>
+            </geometry>
+        </visual>
+        <collision>
+            <origin rpy="0 0 0" xyz="-0.5 -0.5 0"/>
+            <geometry>
+                <mesh filename="package://dexter_description/meshes/basement.STL"
+                      scale="0.01 0.01 0.01"/>
+            </geometry>
+        </collision>
+    </link>
+    <link name="base_plate">
+        <xacro:default_inertial mass="0.1"/>
+        <visual>
+            <origin rpy="0 0 0" xyz="-0.39 -0.39 -0.56"/>
+            <geometry>
+                <mesh filename="package://dexter_description/meshes/base_plate.STL"
+                      scale="0.01 0.01 0.01"/>
+            </geometry>
+        </visual>
+        <collision>
+            <origin rpy="0 0 0" xyz="-0.39 -0.39 -0.56"/>
+            <geometry>
+                <mesh filename="package://dexter_description/meshes/base_plate.STL"
+                      scale="0.01 0.01 0.01"/>
+            </geometry>
+        </collision>
+    </link>
+    <link name="forward_drive_arm">
+        <xacro:default_inertial mass="0.1"/>
+        <visual>
+            <origin rpy=" 0 -${PI / 2} ${PI / 2}" xyz="0.19 0.06 -0.08"/>
+            <geometry>
+                <mesh filename="package://dexter_description/meshes/forward_drive_arm.STL"
+                      scale="0.01 0.01 0.01"/>
+            </geometry>
+        </visual>
+        <collision>
+            <origin rpy=" 0 -${PI / 2} ${PI / 2}" xyz="0.19 0.06 -0.08"/>
+            <geometry>
+                <mesh filename="package://dexter_description/meshes/forward_drive_arm.STL"
+                      scale="0.01 0.01 0.01"/>
+            </geometry>
+        </collision>
+    </link>
+    <link name="horizontal_arm">
+        <xacro:default_inertial mass="0.1"/>
+        <visual>
+            <origin rpy="${PI / 2} 0 ${PI / 2}" xyz="-0.03 -0.4 -0.06"/>
+            <geometry>
+                <mesh filename="package://dexter_description/meshes/horizontal_arm.STL"
+                      scale="0.01 0.01 0.01"/>
+            </geometry>
+        </visual>
+        <collision>
+            <origin rpy="${PI / 2} 0 ${PI / 2}" xyz="-0.03 -0.4 -0.06"/>
+            <geometry>
+                <mesh filename="package://dexter_description/meshes/horizontal_arm.STL"
+                      scale="0.01 0.01 0.01"/>
+            </geometry>
+        </collision>
+    </link>
+    <link name="claw_support">
+        <xacro:default_inertial mass="0.05"/>
+        <visual>
+            <origin rpy="0 0 ${PI / 2}" xyz="0 -0.05 -0.15"/>
+            <geometry>
+                <mesh filename="package://dexter_description/meshes/claw_support.STL"
+                      scale="0.01 0.01 0.01"/>
+            </geometry>
+        </visual>
+        <collision>
+            <origin rpy="0 0 ${PI / 2}" xyz="0 -0.05 -0.15"/>
+            <geometry>
+                <mesh filename="package://dexter_description/meshes/claw_support.STL"
+                      scale="0.01 0.01 0.01"/>
+            </geometry>
+        </collision>
+    </link>
+    <!--
+      gripper_aruco_plate  –  ArUco ID 21, 120×120 mm flat square
+      ─────────────────────────────────────────────────────────────
+      WHY claw_support (not base_plate):
+        • base_plate is occluded by the arm body from above
+        • claw_support is at the gripper TIP — furthest from the base
+          and most exposed to the overhead camera view
+      JOINT PLACEMENT (in claw_support local frame):
+        The claw_support joint connects at horizontal_arm origin + 0.82 m
+        along the arm's local Y axis.
+        The claw_support visual mesh sits at xyz="0 -0.05 -0.15".
+        Joint_4 (gripper_right) is at xyz="-0.04 0.13 -0.1".
+        We place the marker plate at xyz="0 0 0.08" in claw_support
+        frame (8 cm above the joint origin, which is the "top" of the
+        claw body).
+      ORIENTATION (rpy in claw_support frame):
+        When the arm bends toward the shelf (j2≈−0.55, j3≈−1.17),
+        the claw_support's local +Z axis tilts toward world +Z.
+        rpy="0 0 0" makes the marker face the local +Z of claw_support,
+        which aligns roughly with world +Z during picking — exactly when
+        the overhead camera needs to see it.
+      SIZE: 120×120 mm (larger than box markers for better detection at
+      varying heights when arm moves).
+    -->
+    <link name="gripper_aruco_plate">
+        <xacro:default_inertial mass="0.001"/>
+        <visual>
+            <origin xyz="0 0 0" rpy="0 0 0"/>
+            <geometry>
+                <!-- 120×120 mm, 3 mm thick – visually prominent -->
+                <box size="0.12 0.12 0.003"/>
+            </geometry>
+        </visual>
+        <!-- no collision – visual only -->
+    </link>
+    <link name="gripper_right">
+        <xacro:default_inertial mass="0.01"/>
+        <visual>
+            <origin rpy="0 0 -${PI / 2}" xyz="-0.1 0.50 -0.1"/>
+            <geometry>
+                <mesh filename="package://dexter_description/meshes/right_finger.STL"
+                      scale="0.01 0.01 0.01"/>
+            </geometry>
+        </visual>
+        <collision>
+            <origin rpy="0 0 -${PI / 2}" xyz="-0.1 0.50 -0.1"/>
+            <geometry>
+                <mesh filename="package://dexter_description/meshes/right_finger.STL"
+                      scale="0.01 0.01 0.01"/>
+            </geometry>
+        </collision>
+    </link>
+    <link name="gripper_left">
+        <xacro:default_inertial mass="0.01"/>
+        <visual>
+            <origin rpy="0 0 -${PI / 2}" xyz="-0.04 0.50 -0.1"/>
+            <geometry>
+                <mesh filename="package://dexter_description/meshes/left_finger.STL"
+                      scale="0.01 0.01 0.01"/>
+            </geometry>
+        </visual>
+        <collision>
+            <origin rpy="0 0 -${PI / 2}" xyz="-0.04 0.50 -0.1"/>
+            <geometry>
+                <mesh filename="package://dexter_description/meshes/left_finger.STL"
+                      scale="0.01 0.01 0.01"/>
+            </geometry>
+        </collision>
+    </link>
+    <!-- ── Joints ─────────────────────────────────────────────────────────── -->
+    <joint name="virtual_joint" type="fixed">
+        <parent link="world"/>
+        <child  link="base_link"/>
+        <origin xyz="0 0 0" rpy="0 0 0"/>
+    </joint>
+    <joint name="joint_1" type="revolute">
+        <parent link="base_link"/>
+        <child  link="base_plate"/>
+        <origin xyz="0 0 0.307"/>
+        <axis xyz="0 0 1"/>
+        <limit lower="-${PI * 0.95}" upper="${PI * 0.95}"
+               effort="${effort}" velocity="${velocity}"/>
+    </joint>
+    <joint name="joint_2" type="revolute">
+        <parent link="base_plate"/>
+        <child  link="forward_drive_arm"/>
+        <origin xyz="-0.02 0 0.35"/>
+        <axis xyz="1 0 0"/>
+        <limit lower="-${PI / 2}" upper="${PI / 2}"
+               effort="${effort}" velocity="${velocity}"/>
+    </joint>
+    <joint name="joint_3" type="revolute">
+        <parent link="forward_drive_arm"/>
+        <child  link="horizontal_arm"/>
+        <origin xyz="0 0 0.8"/>
+        <axis xyz="1 0 0"/>
+        <limit lower="-${PI / 2}" upper="${PI / 2}"
+               effort="${effort}" velocity="${velocity}"/>
+    </joint>
+    <joint name="horizontal_arm_to_claw_support" type="fixed">
+        <parent link="horizontal_arm"/>
+        <child  link="claw_support"/>
+        <origin xyz="0 0.82 0"/>
+    </joint>
+    <!--
+      gripper_aruco_joint – fixed, attaches the marker plate to claw_support.
+      xyz="0 0 0.08":  8 cm along claw_support local +Z (above the body).
+      rpy="0 0 0":     marker face aligns with claw_support local +Z, which
+                       faces the overhead camera during arm picking motion.
+    -->
+    <joint name="gripper_aruco_joint" type="fixed">
+        <parent link="claw_support"/>
+        <child  link="gripper_aruco_plate"/>
+        <origin xyz="0 0 0.08" rpy="0 0 0"/>
+    </joint>
+    <joint name="joint_4" type="revolute">
+        <parent link="claw_support"/>
+        <child  link="gripper_right"/>
+        <origin xyz="-0.04 0.13 -0.1"/>
+        <axis xyz="0 0 1"/>
+        <limit lower="-${PI / 2}" upper="0.0"
+               effort="${effort}" velocity="${velocity}"/>
+    </joint>
+    <joint name="joint_5" type="revolute">
+        <parent link="claw_support"/>
+        <child  link="gripper_left"/>
+        <origin xyz="-0.22 0.13 -0.1"/>
+        <axis xyz="0 0 1"/>
+        <limit lower="0.0" upper="${PI / 2}"
+               effort="${effort}" velocity="${velocity}"/>
+        <mimic joint="joint_4" multiplier="-1"/>
+    </joint>
+</robot>

File: Dexter/install/dexter_description/share/dexter_description/urdf/dexter_gazebo.xacro (robot description, xacro)
@@ -1 +1,47 @@
-/home/aditya/Cpps/Dexter/dexter_description/urdf/dexter_gazebo.xacro
+<?xml version="1.0"?>
+<robot xmlns:xacro="http://www.ros.org/wiki/xacro" name="dexter">
+  <!-- ── ros2_control plugin ─────────────────────────────────────────────── -->
+  <gazebo>
+    <xacro:if value="$(arg is_ignition)">
+      <plugin filename="ign_ros2_control-system"
+              name="ign_ros2_control::IgnitionROS2ControlPlugin">
+        <parameters>$(find dexter_controller)/config/dexter_controllers.yaml</parameters>
+      </plugin>
+    </xacro:if>
+    <xacro:unless value="$(arg is_ignition)">
+      <plugin filename="gz_ros2_control-system"
+              name="gz_ros2_control::GazeboSimROS2ControlPlugin">
+        <parameters>$(find dexter_controller)/config/dexter_controllers.yaml</parameters>
+      </plugin>
+    </xacro:unless>
+  </gazebo>
+  <!--
+    ── ArUco ID 21 on gripper_aruco_plate (claw_support child) ──────────────
+    This marker is on the TIP of the gripper arm, attached to claw_support.
+    It is visible from the overhead camera when the arm bends toward the shelf
+    (j2≈−0.55, j3≈−1.17) because the top face of claw_support faces upward
+    in that configuration.
+    The detector tracks ID 21 and publishes the gripper world position,
+    which drives closed-loop arm-to-box positioning.
+    PBR settings:
+      metalness=0.0, roughness=1.0 → purely diffuse white background
+      → markers render clearly under the scene lighting in ogre2.
+  -->
+  <gazebo reference="gripper_aruco_plate">
+    <visual name="visual">
+      <cast_shadows>false</cast_shadows>
+      <material>
+        <ambient>1 1 1 1</ambient>
+        <diffuse>1 1 1 1</diffuse>
+        <specular>0 0 0 1</specular>
+        <pbr>
+          <metal>
+            <albedo_map>model://dexter_description/textures/aruco_21.png</albedo_map>
+            <metalness>0.0</metalness>
+            <roughness>1.0</roughness>
+          </metal>
+        </pbr>
+      </material>
+    </visual>
+  </gazebo>
+</robot>

File: Dexter/install/dexter_description/share/dexter_description/urdf/dexter_ros2_control.xacro (robot description, xacro)
@@ -1 +1,60 @@
-/home/aditya/Cpps/Dexter/dexter_description/urdf/dexter_ros2_control.xacro
+<?xml version="1.0"?>
+<robot xmlns:xacro="http://www.ros.org/wiki/xacro" name="dexter">
+    <ros2_control name="RobotSystem" type="system">
+        <xacro:property name="PI" value="3.14159265359" />
+        <!-- ros2_control Gazebo -->
+        <xacro:if value="$(arg is_sim)">
+            <!-- ROS 2 Humble -->
+            <xacro:if value="$(arg is_ignition)">
+                <hardware>
+                    <plugin>ign_ros2_control/IgnitionSystem</plugin>
+                </hardware>
+            </xacro:if>
+            <!-- ROS 2 Iron or above -->
+            <xacro:unless value="$(arg is_ignition)">
+                <hardware>
+                    <plugin>gz_ros2_control/GazeboSimSystem</plugin>
+                </hardware>
+            </xacro:unless>
+            <joint name="joint_5">
+                <param name="mimic">joint_4</param>
+                <param name="multiplier">-1</param>
+            </joint>
+        </xacro:if>
+        <!-- ros2_control Real Robot -->
+        <xacro:unless value="$(arg is_sim)">
+            <hardware>
+                <plugin>dexter_controller/DexterInterface</plugin>
+                <param name="port">/dev/ttyACM0</param>
+            </hardware>
+        </xacro:unless>
+        <joint name="joint_1">
+            <command_interface name="position">
+            <param name="min">-${PI / 2}</param>
+            <param name="max">${PI / 2}</param>
+            </command_interface>
+            <state_interface name="position"/>
+        </joint>
+        <joint name="joint_2">
+            <command_interface name="position">
+            <param name="min">-${PI / 2}</param>
+            <param name="max">${PI / 2}</param>
+            </command_interface>
+            <state_interface name="position"/>
+        </joint>
+        <joint name="joint_3">
+            <command_interface name="position">
+            <param name="min">-${PI / 2}</param>
+            <param name="max">${PI / 2}</param>
+            </command_interface>
+            <state_interface name="position"/>
+        </joint>
+        <joint name="joint_4">
+            <command_interface name="position">
+            <param name="min">-${PI / 2}</param>
+            <param name="max">0.0</param>
+            </command_interface>
+            <state_interface name="position"/>
+        </joint>
+    </ros2_control>
+</robot>
